File: robocar-racer-controller-2026/Car_v1.kicad_sch (KiCad schematic)
At the start: 34 parts, among them J1 GY-87, J10 Buck in, J11 Motor_in, J12 Bateria 3s, J13 Buck_out, J14 Raspbery_usbc, J2 Barramento 16 pinos, J3 Conn_01x03_Pin, J4 Conn_01x03_Pin, J5 Conn_01x19_Socket, J6 Conn_01x19_Socket, J8 ADS1115, J9 Bateria 2s, SW1 SW_DPST_x2, SW2 SW_DPST_x2, U2 ESP32-DEVKITC-32D

Commit message: organizando o esquematico
Parts:
- removed D6: LED_3mm, LED_THT:LED_D3.0mm, symbol PCM_SL_Devices:LED_3mm
- removed J2: Barramento 16 pinos, Connector:SAMTEC_TSW-116-22-T-S, symbol Meus simbolos:Barramento 16 pinos
- added D8: LED_3mm, LED_THT:LED_D3.0mm, symbol PCM_SL_Devices:LED_3mm
- added J15: Step_up, TerminalBlock_Phoenix:TerminalBlock_Phoenix_MKDS-1,5-2-5.08_1x02_P5.08mm_Horizontal, symbol Connector:Screw_Terminal_01x02
- added J16: Radio, Connector_PinHeader_2.54mm:PinHeader_1x04_P2.54mm_Horizontal, symbol Connector:Conn_01x04_Pin
- added J7: Serial, Connector_PinHeader_2.54mm:PinHeader_1x02_P2.54mm_Horizontal, symbol Connector:Conn_01x02_Pin
- J3: value Conn_01x03_Pin -> Sinal_Servo; footprint Connector_PinHeader_2.54mm:PinHeader_1x03_P2.54mm_Vertical -> Connector_PinHeader_2.54mm:PinHeader_1x03_P2.54mm_Horizontal
- J4: value Conn_01x03_Pin -> Sinal_Motor; footprint Connector_PinHeader_2.54mm:PinHeader_1x03_P2.54mm_Vertical -> Connector_PinHeader_2.54mm:PinHeader_1x03_P2.54mm_Horizontal
Connections:
- net RXD0 is gone; now on net RX_RASPBERRY: J5.5 (Pin_5), U2.J3-5 (RXD0)
- net TXD0 is gone; now on net TX_RASPBERRY: J5.4 (Pin_4), U2.J3-4 (TXD0)
- net +12V: now also SW2.2 (B); no longer SW2.1 (A)
- net +5V: now also J16.3 (Pin_3)
- net +8V: now also J15.1 (Pin_1)
- net GND: now also D8.1, J15.2 (Pin_2), J16.4 (Pin_4)
- net Motor Rec: now also J16.2 (Pin_2)
- net RX_RASPBERRY: now also J7.2 (Pin_2)
- net Servo Rec: now also J16.1 (Pin_1)
- net TX_RASPBERRY: now also J7.1 (Pin_1)
- net at J12.2 (Pin_2): now also SW2.1 (A); no longer SW2.2 (B)
- net at R17.2: now also D8.2
- no-connect marks 7 -> 3
Other:
- moved on the sheet: D7, R17, R18, SW2A

Commit message: ajustes na entrada serial
Connections:
- net RX is gone; now on net TX_RASPBERRY: J5.12 (Pin_12), U2.J3-12 (IO16)
- net TX is gone; now on net RX_RASPBERRY: J5.11 (Pin_11), U2.J3-11 (IO17)
- net RX_RASPBERRY: no longer J5.5 (Pin_5), U2.J3-5 (RXD0)
- net TX_RASPBERRY: no longer J5.4 (Pin_4), U2.J3-4 (TXD0)
- new net RXD0: J5.5 (Pin_5), U2.J3-5 (RXD0)
- new net TXD0: J5.4 (Pin_4), U2.J3-4 (TXD0)
Changed lines of the file:
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@@
-	(wire
-		(pts
-			(xy 132.08 135.89) (xy 138.43 135.89)
-		)
-		(stroke
-			(width 0)
-			(type default)
-		)
-	)
 	(wire
 		(pts
@@
 	(wire
 		(pts
+			(xy 132.08 156.21) (xy 135.89 156.21)
+		)
+		(stroke
+			(width 0)
+			(type default)
+		)
+	)
+	(wire
+		(pts
+			(xy 132.08 153.67) (xy 135.89 153.67)
+		)
+		(stroke
+			(width 0)
+			(type default)
+		)
+	)
+	(wire
+		(pts
 			(xy 168.91 116.84) (xy 170.18 116.84)
 		)
@@
 	(wire
 		(pts
+			(xy 133.35 138.43) (xy 132.08 138.43)
+		)
+		(stroke
+			(width 0)
+			(type default)
+		)
+	)
+	(wire
+		(pts
 			(xy 62.23 124.46) (xy 62.23 119.38)
 		)
@@
 	(wire
 		(pts
-			(xy 132.08 138.43) (xy 138.43 138.43)
-		)
-		(stroke
-			(width 0)
-			(type default)
-		)
-	)
-	(wire
-		(pts
 			(xy 168.91 162.56) (xy 170.18 162.56)
 		)
@@
 	(wire
 		(pts
-			(xy 134.62 153.67) (xy 132.08 153.67)
-		)
-		(stroke
-			(width 0)
-			(type default)
-		)
-	)
-	(wire
-		(pts
 			(xy 245.11 127) (xy 246.38 127)
 		)
@@
 	(wire
 		(pts
+			(xy 133.35 135.89) (xy 132.08 135.89)
+		)
+		(stroke
+			(width 0)
+			(type default)
+		)
+	)
+	(wire
+		(pts
 			(xy 36.83 180.34) (xy 34.29 180.34)
 		)
@@
 		(pts
 			(xy 204.47 137.16) (xy 201.93 137.16)
-		)
-		(stroke
-			(width 0)
-			(type default)
-		)
-	)
-	(wire
-		(pts
-			(xy 132.08 156.21) (xy 134.62 156.21)
 		)
 		(stroke
@@
 		)
 	)
-	(label "RXD0"
-		(at 132.08 138.43 0)
-		(effects
-			(font
-				(size 1.27 1.27)
-			)
-			(justify left bottom)
-		)
-	)
 	(label "EN"
 		(at 170.18 119.38 0)
@@
 	)
 	(label "TXD0"
-		(at 132.08 135.89 0)
-		(effects
-			(font
-				(size 1.27 1.27)
-			)
-			(justify left bottom)
-		)
-	)
-	(label "TX"
-		(at 204.47 142.24 0)
+		(at 133.35 135.89 0)
 		(effects
 			(font
@@
 		)
 	)
-	(label "RX"
-		(at 134.62 156.21 0)
-		(effects
-			(font
-				(size 1.27 1.27)
-			)
-			(justify left bottom)
-		)
-	)
 	(label "IO26"
 		(at 91.44 151.13 0)
@@
 		)
 	)
-	(label "TX"
-		(at 134.62 153.67 0)
-		(effects
-			(font
-				(size 1.27 1.27)
-			)
-			(justify left bottom)
-		)
-	)
 	(label "CLK"
 		(at 201.93 162.56 0)
@@
 		)
 	)
+	(label "RXD0"
+		(at 133.35 138.43 0)
+		(effects
+			(font
+				(size 1.27 1.27)
+			)
+			(justify left bottom)
+		)
+	)
 	(label "IO32"
 		(at 170.18 132.08 0)
@@
 	(label "SD0"
 		(at 201.93 160.02 0)
-		(effects
-			(font
-				(size 1.27 1.27)
-			)
-			(justify left bottom)
-		)
-	)
-	(label "RX"
-		(at 204.47 144.78 0)
 		(effects
 			(font
@@
 	(global_label "TX_RASPBERRY"
 		(shape input)
+		(at 204.47 144.78 0)
+		(fields_autoplaced yes)
+		(effects
+			(font
+				(size 1.27 1.27)
+			)
+			(justify left)
+		)
+		(property "Intersheetrefs" "${INTERSHEET_REFS}"
+			(at 221.4856 144.78 0)
+			(hide yes)
+			(show_name no)
+			(do_not_autoplace no)
+			(effects
+				(font
+					(size 1.27 1.27)
+				)
+				(justify left)
+			)
+		)
+	)
+	(global_label "TX_RASPBERRY"
+		(shape input)
 		(at 241.3 60.96 0)
 		(fields_autoplaced yes)
@@
 	(global_label "RX_RASPBERRY"
 		(shape input)
-		(at 138.43 138.43 0)
+		(at 135.89 153.67 0)
 		(fields_autoplaced yes)
 		(effects
@@
 		)
 		(property "Intersheetrefs" "${INTERSHEET_REFS}"
-			(at 155.748 138.43 0)
+			(at 153.208 153.67 0)
 			(hide yes)
 			(show_name no)
@@
 		)
 	)
+	(global_label "RX_RASPBERRY"
+		(shape input)
+		(at 204.47 142.24 0)
+		(fields_autoplaced yes)
+		(effects
+			(font
+				(size 1.27 1.27)
+			)
+			(justify left)
+		)
+		(property "Intersheetrefs" "${INTERSHEET_REFS}"
+			(at 221.788 142.24 0)
+			(hide yes)
+			(show_name no)
+			(do_not_autoplace no)
+			(effects
+				(font
+					(size 1.27 1.27)
+				)
+				(justify left)
+			)
+		)
+	)
 	(global_label "TX_RASPBERRY"
 		(shape input)
-		(at 138.43 135.89 0)
+		(at 135.89 156.21 0)
 		(fields_autoplaced yes)
 		(effects
@@
 		)
 		(property "Intersheetrefs" "${INTERSHEET_REFS}"
-			(at 155.4456 135.89 0)
+			(at 152.9056 156.21 0)
 			(hide yes)
 			(show_name no)
